Commit message: Update kr120r2700.urdf.xacro

File: urdf/kr120r2700.urdf.xacro (robot description, xacro)
@@ -2,5 +2,5 @@
 <robot name="kr120r2700" xmlns:xacro="http://www.ros.org/wiki/xacro">
     <xacro:include filename="$(find kr120)/urdf/macro.xacro"/>
-    <!-- Fix the cobot to the world-->
+    <!-- Fix the robot to the world-->
     <link name="world"/>
     <joint name="fixed" type="fixed">
@@ -8,37 +8,44 @@
         <child link="base_link"/>
     </joint>
-    <xacro:kuka_kr120_r2700 name="base_link" origin_xyz="0.0 0.0 0.0" origin_rpy= "0 0 0"
-                            mass="1" ixx="0.01625" ixy="0" ixz="0" iyy="0.01625" iyz="0" izz="0.005" file_dae="package://kr120/visual/base.dae" file_stl="package://kr120/collision/base.stl"/>
-    <xacro:kuka_kr120_r2700 name="link1" origin_xyz="0.0 0.0 0.0" origin_rpy= "0 0 0"
-                            mass="1.5" ixx="0.054147" ixy="0" ixz="0" iyy="0.054147" iyz="0" izz="0.001875" file_dae="package://kr120/visual/asse1.dae" file_stl="package://kr120/collision/asse1.stl"/>
+    <xacro:kuka_kr120_r2700 name="base_link" origin_xyz="0 0 0" origin_rpy= "0 0 0"
+                            mass="1" ixx="0.01625" ixy="0" ixz="0" iyy="0.01625" iyz="0" izz="0.005" file_dae="package://kr120/visual/base.dae" file_stl="package://kr120/collision/base.stl" scale="0.001 0.001 0.001"/>
+    <xacro:kuka_kr120_r2700 name="link1" origin_xyz="0 0 0" origin_rpy= "0 0 0"
+                            mass="1.5" ixx="0.054147" ixy="0" ixz="0" iyy="0.054147" iyz="0" izz="0.001875" file_dae="package://kr120/visual/asse1.dae" file_stl="package://kr120/collision/asse1.stl" scale="0.001 0.001 0.001"/>
     <xacro:kuka_kr120_r2700_joint name="base_link__link1" type="revolute" parent="base_link" child="link1"
-                            axis="0 0 1" limit_l="-3.14" limit_u="3.14" limit_v="0.5" limit_e="1000"
-                            origin_xyz="0 0 0.05" origin_rpy="0 0 0" />
-    <xacro:kuka_kr120_r2700 name="link2" origin_xyz="0.0 0.0 0.425" origin_rpy= "0 0 0"
-                            mass="2" ixx="0.4816" ixy="0" ixz="0" iyy="0" iyz="0" izz="0.4816" file_dae="package://kr120/visual/asse2.dae" file_stl="package://kr120/collision/asse2.stl"/>
+                            axis="0 0 1" limit_l="-3.22886" limit_u="3.22886" limit_v="2.0944" limit_e="1000"
+                            origin_xyz="0 0 0" origin_rpy="0 0 0" />
+    <xacro:kuka_kr120_r2700 name="link2" origin_xyz="-0.33 0 -0.645" origin_rpy= "0 0 0"
+                            mass="2" ixx="0.4816" ixy="0" ixz="0" iyy="0" iyz="0" izz="0.4816" file_dae="package://kr120/visual/asse2.dae" file_stl="package://kr120/collision/asse2.stl" scale="0.001 0.001 0.001"/>
     <xacro:kuka_kr120_r2700_joint name="link1__link2" type="revolute" parent="link1" child="link2"
-                            axis="0 1 0" limit_l="-2.5" limit_u="2.5" limit_v="0.5" limit_e="1000"
-                            origin_xyz="0 0.1 0.214" origin_rpy="0 0 0" />
-    <xacro:kuka_kr120_r2700 name="link3" origin_xyz="0.0 0.0 0.340" origin_rpy= "0 0 0"
-                            mass="2" ixx="0.4816" ixy="0" ixz="0" iyy="0" iyz="0" izz="0.4816" file_dae="package://kr120/visual/asse3.dae" file_stl="package://kr120/collision/asse3.stl"/>
+                            axis="0 1 0" limit_l="-2.44346" limit_u="-0.0872665" limit_v="2.00713" limit_e="1000"
+                            origin_xyz="0.33 0 0.645" origin_rpy="0 0 0" />
+    <xacro:kuka_kr120_r2700 name="link3" origin_xyz="-0.33 0.0 -1.795" origin_rpy= "0 0 0"
+                            mass="2" ixx="0.4816" ixy="0" ixz="0" iyy="0" iyz="0" izz="0.4816" file_dae="package://kr120/visual/asse3.dae" file_stl="package://kr120/collision/asse3.stl" scale="0.001 0.001 0.001"/>
     <xacro:kuka_kr120_r2700_joint name="link2__link3" type="revolute" parent="link2" child="link3"
-                            axis="0 1 0" limit_l="-3.14" limit_u="3.14" limit_v="0.5" limit_e="1000"
-                            origin_xyz="0 -0.1 0.8" origin_rpy="0 0 0" />
-    <xacro:kuka_kr120_r2700 name="link4" origin_xyz="0.0 0.0 0.065" origin_rpy= "0 0 0"
-                            mass="1" ixx="0.00565" ixy="0" ixz="0" iyy="0" iyz="0" izz="0.00565" file_dae="package://kr120/visual/asse4.dae" file_stl="package://kr120/collision/asse4.stl"/>
+                            axis="0 1 0" limit_l="-2.0944" limit_u="2.93215" limit_v="2.0944" limit_e="1000"
+                            origin_xyz="0 0 1.15" origin_rpy="0 0 0" />
+    <xacro:kuka_kr120_r2700 name="link4" origin_xyz="-0.697 0.0 -1.910" origin_rpy= "0 0 0"
+                            mass="1" ixx="0.00565" ixy="0" ixz="0" iyy="0" iyz="0" izz="0.00565" file_dae="package://kr120/visual/asse4.dae" file_stl="package://kr120/collision/asse4.stl" scale="0.001 0.001 0.001"/>
     <xacro:kuka_kr120_r2700_joint name="link3__link4" type="revolute" parent="link3" child="link4"
-                            axis="0 1 0" limit_l="-3.14" limit_u="3.14" limit_v="0.5" limit_e="1000"
-                            origin_xyz="0 0.1 0.630" origin_rpy="0 0 0" />
-    <xacro:kuka_kr120_r2700 name="link5" origin_xyz="0.0 0.0 0.035" origin_rpy= "0 0 0"
-                            mass="2" ixx="0.4816" ixy="0" ixz="0" iyy="0" iyz="0" izz="0.4816" file_dae="package://kr120/visual/asse5.dae" file_stl="package://kr120/collision/asse5.stl"/>
+                            axis="1 0 0" limit_l="-6.10865" limit_u="6.10865" limit_v="3.31613" limit_e="1000"
+                            origin_xyz="0.367 0 0.115" origin_rpy="0 0 0" />
+    <xacro:kuka_kr120_r2700 name="link5" origin_xyz="-1.55 0 -1.910" origin_rpy= "0 0 0"
+                            mass="2" ixx="0.4816" ixy="0" ixz="0" iyy="0" iyz="0" izz="0.4816" file_dae="package://kr120/visual/asse5.dae" file_stl="package://kr120/collision/asse5.stl" scale="0.001 0.001 0.001"/>
     <xacro:kuka_kr120_r2700_joint name="link4__link5" type="revolute" parent="link4" child="link5"
-                            axis="1 0 0" limit_l="-3.14" limit_u="3.14" limit_v="0.5" limit_e="1000"
-                            origin_xyz="0 0.0 0.180" origin_rpy="0 1.57 0" />
+                            axis="0 1 0" limit_l="-2.18166" limit_u="2.18166" limit_v="3.14159" limit_e="1000"
+                            origin_xyz="0.89 0 0" origin_rpy="0 0 0" />
+    <!-- tool 0 ($FLANGE coordinate system in KRC controller)-->
+    <link name="tool0"/>
     <!-- Build the TCP or end effector-->
-    <xacro:kuka_kr120_r2700 name="flange" origin_xyz="0.0 0.0 0.0" origin_rpy="0 0 0" mass="1"  ixx="0.4816" ixy="0" ixz="0" iyy="0" iyz="0" izz="0.4816"
-                                        file_dae="package://kr120/visual/end-effector.dae" file_stl="package://kr120/collision/end-effector.stl" />
-   <xacro:kuka_kr120_r2700_joint name="link5__flange" type="fixed" parent="link5" child="flange"
-                            axis="1 0 0" limit_l="0" limit_u="0" limit_v="0.5" limit_e="1000"
-                            origin_xyz="0 0.0 0.0" origin_rpy="0 0 0" />
+    <xacro:kuka_kr120_r2700 name="flange" origin_xyz="-1.765 0 -1.910" origin_rpy="0 0 0" mass="1"  ixx="0.4816" ixy="0" ixz="0" iyy="0" iyz="0" izz="0.4816"
+                                        file_dae="package://kr120/visual/end-effector.dae" file_stl="package://kr120/collision/end-effector.stl" scale="0.001 0.001 0.001"/>
+   <xacro:kuka_kr120_r2700_joint name="link5_flange" type="revolute" parent="link5" child="flange"
+                            axis="1 0 0" limit_l="-6.10865" limit_u="6.10865" limit_v="4.53786" limit_e="1000"
+                            origin_xyz="0.215 0 0" origin_rpy="0 0 0" />
+    <joint name="flange__tool0" type="fixed">
+        <origin rpy="0 0 0" xyz="0 0 0"/>
+        <parent link="flange"/>
+        <child link="tool0"/>
+    </joint>
     <!-- put transmission in each joint-->
     <xacro:transmission name="trans_base_link__link1"
@@ -63,5 +70,5 @@
     <gazebo>
         <plugin name="gazebo_ros_control" filename="libgazebo_ros_control.so">
-            <robotNamespace>/kr120r2700</robotNamespace>
+            <robotNamespace>kr120r2700</robotNamespace>
         </plugin>
     </gazebo>
