Commit message: Update macro.xacro

File: urdf/macro.xacro (robot description, xacro)
@@ -16,5 +16,5 @@
             <collision>
                 <geometry>
-                    <mesh filename="${file_stl}/>
+                    <mesh filename="${file_stl}"/>
                 </geometry>
                 <origin xyz="${origin_xyz}" rpy="${origin_rpy}"/>

Commit message: Update macro.xacro

File: urdf/macro.xacro (robot description, xacro)
@@ -1,5 +1,5 @@
 <?xml version = "1.0"?>
 <robot xmlns:xacro="http://www.ros.org/wiki/xacro">
-    <xacro:macro name="kuka_kr120_r2700" params="name origin_xyz origin_rpy mass ixx ixy ixz iyy iyz izz file_dae file_stl">
+    <xacro:macro name="kuka_kr120_r2700" params="name origin_xyz origin_rpy mass ixx ixy ixz iyy iyz izz file_dae file_stl scale">
         <link name="${name}">
             <inertial>
@@ -10,5 +10,5 @@
             <visual>
                 <geometry>
-                    <mesh filename="${file_dae}"/>
+                    <mesh filename="${file_dae}" scale="${scale}"/>
                 </geometry>
                 <origin xyz="${origin_xyz}" rpy="${origin_rpy}"/>
@@ -16,5 +16,5 @@
             <collision>
                 <geometry>
-                    <mesh filename="${file_stl}"/>
+                    <mesh filename="${file_stl}" scale="${scale}"/>
                 </geometry>
                 <origin xyz="${origin_xyz}" rpy="${origin_rpy}"/>

Commit message: Update macro.xacro

File: urdf/macro.xacro (robot description, xacro)
@@ -31,5 +31,5 @@
         </joint>
     </xacro:macro>
-    <xacro:macro name="transmission" params="name joint_name actuator_name">
+    <!--<xacro:macro name="transmission" params="name joint_name actuator_name">
         <transmission name="${name}" >
             <type>transmission_interface/SimpleTransmission</type>
@@ -42,6 +42,6 @@
             </actuator>
         </transmission>
-    </xacro:macro>
-    <xacro:macro name="transmission_effort" params="name joint_name actuator_name">
+    </xacro:macro>-->
+    <xacro:macro name="transmission" params="name joint_name actuator_name">
         <transmission name="${name}" >
             <type>transmission_interface/SimpleTransmission</type>
